File: circuit/device.sch (EAGLE design)
At the start: 11 parts, among them IC1 ATMEGA168-20P, T1 2N2222, T2 2N2222, T3 2N2222, T4 2N2222, T5 2N2222, T6 2N2222, T7 2N2222, T8 2N2222, T9 2N2222

Commit message: added some LEDs and labels
Parts:
- added LED1, LED2: (no value), eagle-ltspice:LED_ELD260
- added R2: 4k7, adafruit:R-US_0204/2V
- added R3, R4: (no value), resistor:R-EU_0204/5
- R1: value (none) -> 4k7
Connections:
- new net +5V: IC1.VCC, R1.2, R2.2
- new net GND: IC1.GND, R3.1, R4.1, T1.E
- new net N$11: LED1.C, R3.2
- new net N$12: IC1.(PCI1/OC1A/OC1S)PB1, LED2.A
- new net SCL: IC1.(PCI13/ADC5/SCL)PC5, R2.1
- new net SDA: IC1.(PCI12/ADC4/SDA)PC4, R1.1, T1.C
- new net SDF: T1.B
- net N$10: now also LED2.C, R4.2; no longer IC1.(PCI12/ADC4/SDA)PC4
- net N$9: now also IC1.(PCI0/ICP/CLKO)PB0, LED1.A; no longer IC1.(PCI13/ADC5/SCL)PC5
Other:
- note added: "I2C audio input line"
- note added: "I2C pull-up resistors"
- moved on the sheet: R1, T1
Changed lines of the file:
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@@
 <layer number="97" name="Info" color="7" fill="1" visible="yes" active="yes"/>
 <layer number="98" name="Guide" color="6" fill="1" visible="yes" active="yes"/>
+<layer number="99" name="SpiceOrder" color="5" fill="1" visible="yes" active="yes"/>
 <layer number="100" name="Muster" color="7" fill="1" visible="no" active="no"/>
 <layer number="101" name="Patch_Top" color="12" fill="4" visible="yes" active="yes"/>
@@
 <parts>
 <part name="IC1" library="adafruit" deviceset="ATMEGA168*P" device="" technology="-20"/>
-<part name="R1" library="adafruit" deviceset="R-US_" device="0204/2V"/>
-<part name="T1" library="adafruit" deviceset="2N2222" device=""/>
+<part name="R1" library="adafruit" deviceset="R-US_" device="0204/2V" value="4k7"/>
 <part name="T2" library="adafruit" deviceset="2N2222" device=""/>
 <part name="T3" library="adafruit" deviceset="2N2222" device=""/>
@@
 <part name="T8" library="adafruit" deviceset="2N2222" device=""/>
 <part name="T9" library="adafruit" deviceset="2N2222" device=""/>
+<part name="R2" library="adafruit" deviceset="R-US_" device="0204/2V" value="4k7"/>
+<part name="GND1" library="supply1" deviceset="GND" device=""/>
+<part name="P+1" library="supply1" deviceset="+5V" device=""/>
+<part name="LED1" library="eagle-ltspice" deviceset="LED_E" device="LD260"/>
+<part name="LED2" library="eagle-ltspice" deviceset="LED_E" device="LD260"/>
+<part name="R3" library="resistor" deviceset="R-EU_" device="0204/5"/>
+<part name="R4" library="resistor" deviceset="R-EU_" device="0204/5"/>
+<part name="GND2" library="supply1" deviceset="GND" device=""/>
+<part name="GND3" library="supply1" deviceset="GND" device=""/>
+<part name="P+2" library="supply1" deviceset="+5V" device=""/>
+<part name="P+3" library="supply1" deviceset="+5V" device=""/>
+<part name="T1" library="adafruit" deviceset="2N2222" device=""/>
+<part name="GND4" library="supply1" deviceset="GND" device=""/>
 </parts>
 <sheets>
 <sheet>
 <plain>
+<text x="116.84" y="30.48" size="1.778" layer="91">I2C pull-up resistors</text>
+<text x="2.54" y="38.1" size="1.778" layer="91">I2C audio input line</text>
 </plain>
 <instances>
 <instance part="IC1" gate="G$1" x="20.32" y="-25.4"/>
-<instance part="R1" gate="G$1" x="60.96" y="27.94"/>
-<instance part="T1" gate="G$1" x="68.58" y="55.88"/>
+<instance part="R1" gate="G$1" x="101.6" y="30.48" rot="R90"/>
 <instance part="T2" gate="G$1" x="119.38" y="-7.62"/>
 <instance part="T3" gate="G$1" x="119.38" y="-20.32"/>
@@
 <instance part="T8" gate="G$1" x="119.38" y="-83.82"/>
 <instance part="T9" gate="G$1" x="119.38" y="-96.52"/>
+<instance part="R2" gate="G$1" x="109.22" y="30.48" rot="R90"/>
+<instance part="GND1" gate="1" x="-7.62" y="-30.48"/>
+<instance part="P+1" gate="1" x="-15.24" y="-33.02"/>
+<instance part="LED1" gate="G$1" x="71.12" y="-71.12"/>
+<instance part="LED2" gate="G$1" x="63.5" y="-71.12"/>
+<instance part="R3" gate="G$1" x="71.12" y="-86.36" rot="R90"/>
+<instance part="R4" gate="G$1" x="63.5" y="-86.36" rot="R90"/>
+<instance part="GND2" gate="1" x="63.5" y="-93.98"/>
+<instance part="GND3" gate="1" x="71.12" y="-93.98"/>
+<instance part="P+2" gate="1" x="109.22" y="40.64"/>
+<instance part="P+3" gate="1" x="101.6" y="40.64"/>
+<instance part="T1" gate="G$1" x="-15.24" y="35.56" rot="MR0"/>
+<instance part="GND4" gate="1" x="-17.78" y="27.94"/>
 </instances>
 <busses>
@@
 </segment>
 </net>
-<net name="N$9" class="0">
+<net name="SCL" class="0">
 <segment>
 <pinref part="IC1" gate="G$1" pin="(PCI13/ADC5/SCL)PC5"/>
 <wire x1="53.34" y1="-10.16" x2="83.82" y2="-10.16" width="0.1524" layer="91"/>
-<wire x1="83.82" y1="-10.16" x2="83.82" y2="20.32" width="0.1524" layer="91"/>
-</segment>
-</net>
-<net name="N$10" class="0">
+<wire x1="83.82" y1="-10.16" x2="83.82" y2="15.24" width="0.1524" layer="91"/>
+<wire x1="83.82" y1="15.24" x2="109.22" y2="15.24" width="0.1524" layer="91"/>
+<label x="119.38" y="15.24" size="1.778" layer="95"/>
+<pinref part="R2" gate="G$1" pin="1"/>
+<wire x1="109.22" y1="15.24" x2="124.46" y2="15.24" width="0.1524" layer="91"/>
+<wire x1="109.22" y1="25.4" x2="109.22" y2="15.24" width="0.1524" layer="91"/>
+<junction x="109.22" y="15.24"/>
+</segment>
+</net>
+<net name="SDA" class="0">
 <segment>
 <pinref part="IC1" gate="G$1" pin="(PCI12/ADC4/SDA)PC4"/>
 <wire x1="53.34" y1="-7.62" x2="81.28" y2="-7.62" width="0.1524" layer="91"/>
-<wire x1="81.28" y1="-7.62" x2="81.28" y2="20.32" width="0.1524" layer="91"/>
-</segment>
-</net>
+<wire x1="81.28" y1="-7.62" x2="81.28" y2="17.78" width="0.1524" layer="91"/>
+<wire x1="81.28" y1="17.78" x2="101.6" y2="17.78" width="0.1524" layer="91"/>
+<label x="119.38" y="17.78" size="1.778" layer="95"/>
+<pinref part="R1" gate="G$1" pin="1"/>
+<wire x1="101.6" y1="17.78" x2="124.46" y2="17.78" width="0.1524" layer="91"/>
+<wire x1="101.6" y1="25.4" x2="101.6" y2="17.78" width="0.1524" layer="91"/>
+<junction x="101.6" y="17.78"/>
+</segment>
+<segment>
+<pinref part="T1" gate="G$1" pin="C"/>
+<wire x1="-17.78" y1="40.64" x2="-17.78" y2="45.72" width="0.1524" layer="91"/>
+<wire x1="-17.78" y1="45.72" x2="-25.4" y2="45.72" width="0.1524" layer="91"/>
+<label x="-25.4" y="45.72" size="1.778" layer="95"/>
+</segment>
+</net>
+<net name="GND" class="0">
+<segment>
+<pinref part="IC1" gate="G$1" pin="GND"/>
+<wire x1="-2.54" y1="-27.94" x2="-7.62" y2="-27.94" width="0.1524" layer="91"/>
+<pinref part="GND1" gate="1" pin="GND"/>
+</segment>
+<segment>
+<pinref part="R4" gate="G$1" pin="1"/>
+<pinref part="GND2" gate="1" pin="GND"/>
+</segment>
+<segment>
+<pinref part="R3" gate="G$1" pin="1"/>
+<pinref part="GND3" gate="1" pin="GND"/>
+</segment>
+<segment>
+<pinref part="T1" gate="G$1" pin="E"/>
+<pinref part="GND4" gate="1" pin="GND"/>
+</segment>
+</net>
+<net name="N$9" class="0">
+<segment>
+<pinref part="IC1" gate="G$1" pin="(PCI0/ICP/CLKO)PB0"/>
+<wire x1="53.34" y1="-45.72" x2="71.12" y2="-45.72" width="0.1524" layer="91"/>
+<wire x1="71.12" y1="-45.72" x2="71.12" y2="-68.58" width="0.1524" layer="91"/>
+<pinref part="LED1" gate="G$1" pin="A"/>
+</segment>
+</net>
+<net name="N$10" class="0">
+<segment>
+<pinref part="LED2" gate="G$1" pin="C"/>
+<pinref part="R4" gate="G$1" pin="2"/>
+<wire x1="63.5" y1="-76.2" x2="63.5" y2="-81.28" width="0.1524" layer="91"/>
+</segment>
+</net>
+<net name="N$11" class="0">
+<segment>
+<pinref part="LED1" gate="G$1" pin="C"/>
+<pinref part="R3" gate="G$1" pin="2"/>
+<wire x1="71.12" y1="-76.2" x2="71.12" y2="-81.28" width="0.1524" layer="91"/>
+</segment>
+</net>
+<net name="N$12" class="0">
+<segment>
+<pinref part="LED2" gate="G$1" pin="A"/>
+<wire x1="63.5" y1="-68.58" x2="63.5" y2="-48.26" width="0.1524" layer="91"/>
+<pinref part="IC1" gate="G$1" pin="(PCI1/OC1A/OC1S)PB1"/>
+<wire x1="63.5" y1="-48.26" x2="53.34" y2="-48.26" width="0.1524" layer="91"/>
+</segment>
+</net>
+<net name="+5V" class="0">
+<segment>
+<pinref part="P+1" gate="1" pin="+5V"/>
+<wire x1="-15.24" y1="-35.56" x2="-2.54" y2="-35.56" width="0.1524" layer="91"/>
+<pinref part="IC1" gate="G$1" pin="VCC"/>
+<wire x1="-2.54" y1="-35.56" x2="-2.54" y2="-33.02" width="0.1524" layer="91"/>
+</segment>
+<segment>
+<pinref part="R2" gate="G$1" pin="2"/>
+<wire x1="109.22" y1="35.56" x2="109.22" y2="38.1" width="0.1524" layer="91"/>
+<pinref part="P+2" gate="1" pin="+5V"/>
+</segment>
+<segment>
+<pinref part="R1" gate="G$1" pin="2"/>
+<wire x1="101.6" y1="35.56" x2="101.6" y2="38.1" width="0.1524" layer="91"/>
+<pinref part="P+3" gate="1" pin="+5V"/>
+</segment>
+</net>
+<net name="SDF" class="0">
+<segment>
+<wire x1="-12.7" y1="35.56" x2="2.54" y2="35.56" width="0.1524" layer="91"/>
+<pinref part="T1" gate="G$1" pin="B"/>
+</segment>
+</net>

Commit message: playing around in ealge
Parts:
- added LED3: (no value), eagle-ltspice:LED_ELD260
- added R5: (no value), resistor:R-EU_0204/5
Connections:
- net N$12 renamed PB1
- new net PB0: IC1.(PCI0/ICP/CLKO)PB0, LED3.A
- new net PB2: IC1.(PCI2/SS/OC1B)PB2, LED1.A
- new net PB3: IC1.(PCI3/MOSI/OC2A)PB3
- net GND: now also R5.1
- net N$9: now also LED3.C, R5.2; no longer IC1.(PCI0/ICP/CLKO)PB0, LED1.A
Other:
- moved on the sheet: LED1, LED2, R3, R4
Changed lines of the file:
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@@
 <?xml version="1.0" encoding="utf-8"?>
 <!DOCTYPE eagle SYSTEM "eagle.dtd">
-<eagle version="6.4">
+<eagle version="6.5.0">
 <drawing>
 <settings>
@@
 <layer number="97" name="Info" color="7" fill="1" visible="yes" active="yes"/>
 <layer number="98" name="Guide" color="6" fill="1" visible="yes" active="yes"/>
-<layer number="99" name="SpiceOrder" color="5" fill="1" visible="yes" active="yes"/>
+<layer number="99" name="SpiceOrder" color="5" fill="1" visible="no" active="yes"/>
 <layer number="100" name="Muster" color="7" fill="1" visible="no" active="no"/>
 <layer number="101" name="Patch_Top" color="12" fill="4" visible="yes" active="yes"/>
@@
 <part name="R3" library="resistor" deviceset="R-EU_" device="0204/5"/>
 <part name="R4" library="resistor" deviceset="R-EU_" device="0204/5"/>
-<part name="GND2" library="supply1" deviceset="GND" device=""/>
 <part name="GND3" library="supply1" deviceset="GND" device=""/>
 <part name="P+2" library="supply1" deviceset="+5V" device=""/>
@@
 <part name="T1" library="adafruit" deviceset="2N2222" device=""/>
 <part name="GND4" library="supply1" deviceset="GND" device=""/>
+<part name="LED3" library="eagle-ltspice" deviceset="LED_E" device="LD260"/>
+<part name="GND2" library="supply1" deviceset="GND" device=""/>
+<part name="R5" library="resistor" deviceset="R-EU_" device="0204/5"/>
+<part name="GND5" library="supply1" deviceset="GND" device=""/>
 </parts>
 <sheets>
@@
 <instance part="GND1" gate="1" x="-7.62" y="-30.48"/>
 <instance part="P+1" gate="1" x="-15.24" y="-33.02"/>
-<instance part="LED1" gate="G$1" x="71.12" y="-71.12"/>
-<instance part="LED2" gate="G$1" x="63.5" y="-71.12"/>
-<instance part="R3" gate="G$1" x="71.12" y="-86.36" rot="R90"/>
-<instance part="R4" gate="G$1" x="63.5" y="-86.36" rot="R90"/>
-<instance part="GND2" gate="1" x="63.5" y="-93.98"/>
-<instance part="GND3" gate="1" x="71.12" y="-93.98"/>
+<instance part="LED1" gate="G$1" x="38.1" y="-99.06"/>
+<instance part="LED2" gate="G$1" x="22.86" y="-99.06"/>
+<instance part="R3" gate="G$1" x="38.1" y="-111.76" rot="R90"/>
+<instance part="R4" gate="G$1" x="22.86" y="-111.76" rot="R90"/>
+<instance part="GND3" gate="1" x="38.1" y="-121.92"/>
 <instance part="P+2" gate="1" x="109.22" y="40.64"/>
 <instance part="P+3" gate="1" x="101.6" y="40.64"/>
 <instance part="T1" gate="G$1" x="-15.24" y="35.56" rot="MR0"/>
 <instance part="GND4" gate="1" x="-17.78" y="27.94"/>
+<instance part="LED3" gate="G$1" x="7.62" y="-99.06"/>
+<instance part="GND2" gate="1" x="22.86" y="-121.92"/>
+<instance part="R5" gate="G$1" x="7.62" y="-111.76" rot="R90"/>
+<instance part="GND5" gate="1" x="7.62" y="-121.92"/>
 </instances>
 <busses>
@@
 </segment>
 <segment>
-<pinref part="R4" gate="G$1" pin="1"/>
-<pinref part="GND2" gate="1" pin="GND"/>
-</segment>
-<segment>
 <pinref part="R3" gate="G$1" pin="1"/>
 <pinref part="GND3" gate="1" pin="GND"/>
+<wire x1="38.1" y1="-116.84" x2="38.1" y2="-119.38" width="0.1524" layer="91"/>
 </segment>
 <segment>
@@
 <pinref part="GND4" gate="1" pin="GND"/>
 </segment>
-</net>
-<net name="N$9" class="0">
-<segment>
-<pinref part="IC1" gate="G$1" pin="(PCI0/ICP/CLKO)PB0"/>
-<wire x1="53.34" y1="-45.72" x2="71.12" y2="-45.72" width="0.1524" layer="91"/>
-<wire x1="71.12" y1="-45.72" x2="71.12" y2="-68.58" width="0.1524" layer="91"/>
-<pinref part="LED1" gate="G$1" pin="A"/>
+<segment>
+<pinref part="R4" gate="G$1" pin="1"/>
+<wire x1="22.86" y1="-116.84" x2="22.86" y2="-119.38" width="0.1524" layer="91"/>
+<pinref part="GND2" gate="1" pin="GND"/>
+</segment>
+<segment>
+<pinref part="R5" gate="G$1" pin="1"/>
+<pinref part="GND5" gate="1" pin="GND"/>
+<wire x1="7.62" y1="-116.84" x2="7.62" y2="-119.38" width="0.1524" layer="91"/>
 </segment>
 </net>
@@
 <pinref part="LED2" gate="G$1" pin="C"/>
 <pinref part="R4" gate="G$1" pin="2"/>
-<wire x1="63.5" y1="-76.2" x2="63.5" y2="-81.28" width="0.1524" layer="91"/>
+<wire x1="22.86" y1="-104.14" x2="22.86" y2="-106.68" width="0.1524" layer="91"/>
 </segment>
 </net>
@@
 <pinref part="LED1" gate="G$1" pin="C"/>
 <pinref part="R3" gate="G$1" pin="2"/>
-<wire x1="71.12" y1="-76.2" x2="71.12" y2="-81.28" width="0.1524" layer="91"/>
-</segment>
-</net>
-<net name="N$12" class="0">
-<segment>
-<pinref part="LED2" gate="G$1" pin="A"/>
-<wire x1="63.5" y1="-68.58" x2="63.5" y2="-48.26" width="0.1524" layer="91"/>
-<pinref part="IC1" gate="G$1" pin="(PCI1/OC1A/OC1S)PB1"/>
-<wire x1="63.5" y1="-48.26" x2="53.34" y2="-48.26" width="0.1524" layer="91"/>
+<wire x1="38.1" y1="-104.14" x2="38.1" y2="-106.68" width="0.1524" layer="91"/>
 </segment>
 </net>
@@
 </segment>
 </net>
+<net name="N$9" class="0">
+<segment>
+<pinref part="R5" gate="G$1" pin="2"/>
+<pinref part="LED3" gate="G$1" pin="C"/>
+<wire x1="7.62" y1="-106.68" x2="7.62" y2="-104.14" width="0.1524" layer="91"/>
+</segment>
+</net>
+<net name="PB0" class="0">
+<segment>
+<pinref part="IC1" gate="G$1" pin="(PCI0/ICP/CLKO)PB0"/>
+<wire x1="53.34" y1="-45.72" x2="58.42" y2="-45.72" width="0.1524" layer="91"/>
+</segment>
+<segment>
+<pinref part="LED3" gate="G$1" pin="A"/>
+<wire x1="7.62" y1="-96.52" x2="7.62" y2="-88.9" width="0.1524" layer="91"/>
+<label x="7.62" y="-88.9" size="1.778" layer="95"/>
+</segment>
+</net>
+<net name="PB1" class="0">
+<segment>
+<pinref part="IC1" gate="G$1" pin="(PCI1/OC1A/OC1S)PB1"/>
+<wire x1="53.34" y1="-48.26" x2="58.42" y2="-48.26" width="0.1524" layer="91"/>
+</segment>
+<segment>
+<pinref part="LED2" gate="G$1" pin="A"/>
+<wire x1="22.86" y1="-96.52" x2="22.86" y2="-88.9" width="0.1524" layer="91"/>
+<label x="22.86" y="-88.9" size="1.778" layer="95"/>
+</segment>
+</net>
+<net name="PB2" class="0">
+<segment>
+<pinref part="IC1" gate="G$1" pin="(PCI2/SS/OC1B)PB2"/>
+<wire x1="53.34" y1="-50.8" x2="58.42" y2="-50.8" width="0.1524" layer="91"/>
+</segment>
+<segment>
+<pinref part="LED1" gate="G$1" pin="A"/>
+<wire x1="38.1" y1="-96.52" x2="38.1" y2="-88.9" width="0.1524" layer="91"/>
+<label x="38.1" y="-88.9" size="1.778" layer="95"/>
+</segment>
+</net>
+<net name="PB3" class="0">
+<segment>
+<pinref part="IC1" gate="G$1" pin="(PCI3/MOSI/OC2A)PB3"/>
+<wire x1="53.34" y1="-53.34" x2="58.42" y2="-53.34" width="0.1524" layer="91"/>
+</segment>
+</net>
